File: scanner_schematic/scanner_schematic.kicad_sch (KiCad schematic)
At the start: 7 parts, among them M1 Motor_Servo, M2 Motor_Servo, SW1 SW_Push, U1 GP2Y0A02YK0F

Commit message: Clean up schematic
Parts:
- BT1: value Battery -> External Power Supply
Other:
- note added: "Distance Sensor"
- moved on the sheet: BT1, M1, M2, R1, SW1
